File: electronic/pcb1.kicad_pcb (KiCad board)
At the start: 2 copper layers, 24 parts, among them J1 Conn_01x12, U1 AP1509-3SG-13, U2 MAX3232CDR, U3 SparkfunM9N, U4 SN65HVD234, U5 ESP32-WROOM-32U

Commit message: Creation
Parts:
- added D3: D_Schottky, Diode_SMD:D_SMA, F.Cu at (151.1, 110.5)
- added FB1: 100MHz 6A, Resistor_SMD:R_1206_3216Metric, F.Cu at (151.3, 115.6)
- C1: value tantalum_470uF_30V_polarized -> 470UF; footprint Capacitor_SMD:CP_Elec_8x10 -> Capacitor_SMD:CP_Elec_10x10
- C2, C3, C4, C5: value 0,1uF -> 0.1uF
- C6: value tantalum_270uF_10V_polarized -> 330uF; footprint Capacitor_Tantalum_SMD:CP_EIA-3528-21_Kemet-B -> Capacitor_SMD:CP_Elec_10x10
- D2: value WE_155301BS73100 -> Green
- JP1: value SolderJumper_3_Open -> MOSI/RX; moved to B.Cu
- JP2: value SolderJumper_3_Open -> MISO/TX; moved to B.Cu
- L1: value 68uH -> 47uH; footprint Inductor_SMD:L_1210_3225Metric -> Inductor_SMD:L_0805_2012Metric_Pad1.15x1.40mm_HandSolder
- R1: value 250ohm -> 220ohm
- U1: value AP1509-3SG-13 -> XLSEMI XL1509-3.3E1
- U2: footprint Package_SO:SSOP-16_5.3x6.2mm_P0.65mm -> Package_SO:SOIC-16_3.9x9.9mm_P1.27mm
- U4: value SN65HVD234 -> SN65HVD232DR
- U5: footprint RF_Module:ESP32-WROOM-32 -> RF_Module:ESP32-WROOM-32U
- moved C8 77.4 mm to (109.2, 109.2), turned to 270 degrees
- moved C3 54.5 mm to (133.3, 85.1), turned to 90 degrees
- moved U4 50.3 mm to (138.4, 100.3)
- moved C2 47.8 mm to (135.9, 91.9), turned to 90 degrees
- moved U2 47.6 mm to (139.7, 85.1), turned to 90 degrees
- moved J1 46.4 mm to (158.8, 104.1), turned to 90 degrees
- moved U5 46.4 mm to (120.7, 90.2), turned to 90 degrees
- moved JP1 44.9 mm to (120.7, 72.4), turned to 180 degrees
- moved R1 42.9 mm to (158.8, 109.2)
- moved C7 41.8 mm to (135.9, 78.7), turned to 90 degrees
- moved C6 41.5 mm to (116.7, 113.0), turned to 180 degrees
- moved JP2 41.0 mm to (120.7, 76.2)
- moved L1 40.7 mm to (125.7, 109.2), turned to 180 degrees
- moved R2 38.2 mm to (133.3, 78.7), turned to 270 degrees
- moved C9 37.3 mm to (109.2, 116.8), turned to 90 degrees
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Connections:
- net I2C_SCL renamed /I2C_P
- net I2C_SDA renamed /I2C_N
- C1 pad 1: +BATT -> Net-(C1-Pad1)
- C3 pad 1: GND -> Net-(C3-Pad1)
- C3 pad 2: Net-(C3-Pad2) -> GND
- C4 pad 1: GND -> Net-(C4-Pad1)
- C4 pad 2: Net-(C4-Pad2) -> GND
- D2 pad 1: /ESP_LED_CTRL -> Net-(D2-Pad1)
- D2 pad 2: Net-(D2-Pad2) -> /ESP_LED_CTRL
- J1 pad 10: CAN_H -> /RX_FLASH
- J1 pad 11: Net-(J1-Pad11) -> /TX_FLASH
- J1 pad 3: /RX_FLASH -> Net-(J1-Pad3)
- J1 pad 4: /TX_FLASH -> /CAN_N
- J1 pad 5: /RX_UART1 -> /CAN_P
- J1 pad 6: /TX_UART1 -> /RX232_TX2
- J1 pad 7: /TX_UART2 -> /RX232_RX2
- J1 pad 8: /RX_UART2 -> /RX232_RX1
- J1 pad 9: CAN_L -> /RS232_TX1
- R1 pad 2: Net-(D2-Pad2) -> Net-(D2-Pad1)
- R3 pad 1: CAN_L -> /CAN_N
- R3 pad 2: Net-(J1-Pad11) -> Net-(J1-Pad3)
- U1 pad 1: +BATT -> Net-(C1-Pad1)
- U2 pad 13: RS232_RX1 -> /RX232_RX1
- U2 pad 14: RS232_TX1 -> /RS232_TX1
- U2 pad 2: Net-(C3-Pad2) -> Net-(C3-Pad1)
- U2 pad 6: Net-(C4-Pad2) -> Net-(C4-Pad1)
- U2 pad 7: RS232_TX2 -> /RX232_TX2
- U2 pad 8: RS232_RX2 -> /RX232_RX2
- U4 pad 1: CANTX -> /CANX_P
- U4 pad 4: CANRX -> /CANX_N
- U4 pad 5: +3V3 -> Net-(U4-Pad5)
- U4 pad 6: CAN_L -> /CAN_N
- U4 pad 7: CAN_H -> /CAN_P
- U4 pad 8: GND -> Net-(U4-Pad8)
- U5 pad 10: CANRX -> /RX_UART2
- U5 pad 11: CANTX -> /TX_UART2
- U5 pad 27: /RX_UART2 -> /CANX_N
- U5 pad 28: /TX_UART2 -> /CANX_P
Routing:
- net GND: track 0.00 -> 159.4 mm, vias 0 -> 13
- net SPI_CS: track 0.00 -> 125.1 mm, vias 0 -> 1
- net +3V3: track 0.00 -> 120.2 mm, vias 0 -> 3
- net /TX_UART2: track 0.00 -> 112.5 mm, vias 0 -> 2
- net /RX_UART2: track 0.00 -> 108.9 mm, vias 0 -> 2
- net GPS_RX: track 0.00 -> 55.5 mm, vias 0 -> 1
- net /I2C_P: track 0.00 -> 53.9 mm, vias 0 -> 1
- net /GPIO0: track 0.00 -> 50.5 mm, vias 0 -> 2
- net /ESP_LED_CTRL: track 0.00 -> 49.4 mm, vias 0 -> 2
- net /TX_FLASH: track 0.00 -> 48.2 mm, vias 0 -> 1
- net /RX_FLASH: track 0.00 -> 46.1 mm, vias 0 -> 1
- net /I2C_N: track 0.00 -> 43.9 mm, vias 0 -> 1
- net SPI_MOSI: track 0.00 -> 37.8 mm, vias 0 -> 1
- net SPI_SCK: track 0.00 -> 36.6 mm
- net SPI_MISO: track 0.00 -> 35.8 mm, vias 0 -> 1
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- added copper zone on F.Cu, net +3V3
- added copper zone on B.Cu, net GND
Other:
- board outline added: 58.4 x 50.8 mm
- board text added: "SPI / UART"
- board text added: "UART / SPI"
- board text added: "XtraLarge GPS N2K Wifi V1.0"
