File: electronic/pcb1.sch (KiCad schematic (older format))
At the start: 24 parts, among them J1 Conn_01x12, U1 AP1509-3SG-13, U2 MAX3232CDR, U3 SparkfunM9N, U4 SN65HVD234, U5 ESP32-WROOM-32U

Commit message: Creation
Parts:
- removed C2, C3, C4, C5: 0,1uF, Capacitor_SMD:C_0603_1608Metric, symbol pcb1-rescue:C-Device
- added C2, C3, C4, C5: 0.1uF, Capacitor_SMD:C_0603_1608Metric, symbol Device:C
- added D3: D_Schottky, Diode_SMD:D_SMA, symbol Device:D_Schottky
- added FB1: 100MHz 6A, Resistor_SMD:R_1206_3216Metric, symbol Device:Ferrite_Bead
- C1: value tantalum_470uF_30V_polarized -> 470UF; footprint Capacitor_SMD:CP_Elec_8x10 -> Capacitor_SMD:CP_Elec_10x10; symbol pcb1-rescue:CP1-Device -> Device:CP; LCSC C164065 -> C249931; MFR (none) -> VE-471M1ETR-1010
- C6: value tantalum_270uF_10V_polarized -> 330uF; footprint Capacitor_Tantalum_SMD:CP_EIA-3528-21_Kemet-B -> Capacitor_SMD:CP_Elec_10x10; symbol pcb1-rescue:CP1-Device -> Device:CP; LCSC C16133 -> C134522; MFR (none) -> VZH331M1VTR-1010K
- C7: symbol pcb1-rescue:C-Device -> Device:C; MFR (none) -> CC0603KRX7R9BB104
- C8: symbol pcb1-rescue:C-Device -> Device:C; LCSC C19702 -> C15525; MFR (none) -> CL05A106MQ5NUNC
- C9: symbol pcb1-rescue:C-Device -> Device:C; MFR (none) -> CL10A225KO8NNNC
- D1: symbol pcb1-rescue:D_Schottky-Device -> Device:D_Schottky; MFR (none) -> B5819W
- D2: value WE_155301BS73100 -> Green; symbol pcb1-rescue:LED-Device -> Device:LED; LCSC (none) -> C72043; MFR (none) -> 19-217/GHC-YR1S2/3T
- J1: symbol pcb1-rescue:Conn_01x12-Connector_Generic -> Connector_Generic:Conn_01x12
- JP1: value SolderJumper_3_Open -> MOSI/RX; symbol pcb1-rescue:SolderJumper_3_Open-Jumper -> Jumper:SolderJumper_3_Open
- JP2: value SolderJumper_3_Open -> MISO/TX; symbol pcb1-rescue:SolderJumper_3_Open-Jumper -> Jumper:SolderJumper_3_Open
- L1: value 68uH -> 47uH; footprint Inductor_SMD:L_1210_3225Metric -> Inductor_SMD:L_0805_2012Metric_Pad1.15x1.40mm_HandSolder; symbol pcb1-rescue:L-Device -> Device:L_Small; LCSC C76843 -> C14304; MFR (none) -> SDFL2012T470KTF
- R1: value 250ohm -> 220ohm; symbol pcb1-rescue:R-Device -> Device:R; MFR (none) -> 0402WGF2200TCE
- R2, R4: symbol pcb1-rescue:R-Device -> Device:R; MFR (none) -> 0603WAF1002T5E
- R3: symbol pcb1-rescue:R-Device -> Device:R; LCSC C25804 -> C25205; MFR (none) -> 0603WAJ0121T5E
- U1: value AP1509-3SG-13 -> XLSEMI XL1509-3.3E1; LCSC (none) -> C74193; MFR (none) -> XL1509-3.3E1
- U2: footprint Package_SO:SSOP-16_5.3x6.2mm_P0.65mm -> Package_SO:SOIC-16_3.9x9.9mm_P1.27mm; symbol pcb1-rescue:MAX3232-Interface_UART -> Interface_UART:MAX3232; LCSC (none) -> C45843; MFR (none) -> MAX3232CDR
- U4: value SN65HVD234 -> SN65HVD232DR; symbol pcb1-rescue:SN65HVD234-Interface_CAN_LIN -> Interface_CAN_LIN:SN65HVD232; LCSC (none) -> C30530; MFR (none) -> SN65HVD232DR
- U5: footprint RF_Module:ESP32-WROOM-32 -> RF_Module:ESP32-WROOM-32U; symbol pcb1-rescue:ESP32-WROOM-32U-RF_Module -> RF_Module:ESP32-WROOM-32U; LCSC (none) -> C529580; MFR (none) -> ESP32-WROOM-32U(16MB)
Connections:
- net labels added: CANX_N, CANX_P, CAN_N, CAN_P, I2C_N, I2C_P, RX232_RX1, RX232_RX2, RX232_TX2
- net labels removed: CANRX, CANTX, CAN_H, CAN_L, I2C_SCL, I2C_SDA, RS232_RX1, RS232_RX2, RS232_TX2
- wire segments 71 -> 95

Commit message: Version 1.0 proto commande JLCPCB
Parts:
- U1: symbol pcb1-rescue:AP1509-50SG-13-Converter_DCDC -> pcb1-rescue:AP1509-50SG-13-Converter_DCDC-pcb1-rescue
- U3: symbol pcb1-rescue:SparkfunM9N-sparkfunm9n -> pcb1-rescue:SparkfunM9N-sparkfunm9n-pcb1-rescue
Changed lines of the file:
@@
 GPIO0
 $Comp
-L pcb1-rescue:GND-power #PWR021
+L pcb1-rescue:GND-power-pcb1-rescue #PWR021
 U 1 1 5EAAA240
 P 9150 4900
@@
 	650  2750 3450 2750
 $Comp
-L pcb1-rescue:+3.3V-power #PWR011
+L pcb1-rescue:+3.3V-power-pcb1-rescue #PWR011
 U 1 1 5EB0540C
 P 4900 1600
@@
 $EndComp
 $Comp
-L pcb1-rescue:+3.3V-power #PWR014
+L pcb1-rescue:+3.3V-power-pcb1-rescue #PWR014
 U 1 1 5EB07502
 P 6100 3050
@@
 	6100 3100 6100 3050
 $Comp
-L pcb1-rescue:+3.3V-power #PWR022
+L pcb1-rescue:+3.3V-power-pcb1-rescue #PWR022
 U 1 1 5EB151FE
 P 10650 1650
@@
 $EndComp
 $Comp
-L pcb1-rescue:+BATT-power #PWR018
+L pcb1-rescue:+BATT-power-pcb1-rescue #PWR018
 U 1 1 5EB20F66
 P 6650 1600
@@
 $EndComp
 $Comp
-L pcb1-rescue:PWR_FLAG-power #FLG01
+L pcb1-rescue:PWR_FLAG-power-pcb1-rescue #FLG01
 U 1 1 5EB2CD1E
 P 6650 1600
@@
 $EndComp
 $Comp
-L pcb1-rescue:GND-power #PWR015
+L pcb1-rescue:GND-power-pcb1-rescue #PWR015
 U 1 1 5EA7B173
 P 6100 4000
@@
 	1000 1650 1000 1900
 $Comp
-L pcb1-rescue:+BATT-power #PWR01
+L pcb1-rescue:+BATT-power-pcb1-rescue #PWR01
 U 1 1 5EB287B8
 P 800 700
@@
 	2700 1650 2700 1750
 $Comp
-L pcb1-rescue:GND-power #PWR02
+L pcb1-rescue:GND-power-pcb1-rescue #PWR02
 U 1 1 5EC64914
 P 1550 2450
@@
 	3250 1650 3250 1700
 $Comp
-L pcb1-rescue:AP1509-50SG-13-Converter_DCDC U1
+L pcb1-rescue:AP1509-50SG-13-Converter_DCDC-pcb1-rescue U1
 U 1 1 5FBB15D5
 P 2000 1750
@@
 SPI_MISO
 $Comp
-L pcb1-rescue:SparkfunM9N-sparkfunm9n U3
+L pcb1-rescue:SparkfunM9N-sparkfunm9n-pcb1-rescue U3
 U 1 1 5FC757E9
 P 4950 5450
@@
 $EndComp
 $Comp
-L pcb1-rescue:GND-power #PWR012
+L pcb1-rescue:GND-power-pcb1-rescue #PWR012
 U 1 1 5FC7624D
 P 5650 5100
@@
 	2800 4350 3100 4350
 $Comp
-L pcb1-rescue:GND-power #PWR06
+L pcb1-rescue:GND-power-pcb1-rescue #PWR06
 U 1 1 5FCC18BF
 P 3400 4700
@@
 Connection ~ 3400 4700
 $Comp
-L pcb1-rescue:GND-power #PWR03
+L pcb1-rescue:GND-power-pcb1-rescue #PWR03
 U 1 1 5FCCB5E0
 P 2000 6150
@@
 TX_UART1
 $Comp
-L pcb1-rescue:+3.3V-power #PWR05
+L pcb1-rescue:+3.3V-power-pcb1-rescue #PWR05
 U 1 1 5FCDA3FC
 P 3250 850
@@
 $EndComp
 $Comp
-L pcb1-rescue:GND-power #PWR017
+L pcb1-rescue:GND-power-pcb1-rescue #PWR017
 U 1 1 5EA85535
 P 6550 1600
@@
 $EndComp
 $Comp
-L pcb1-rescue:GND-power #PWR019
+L pcb1-rescue:GND-power-pcb1-rescue #PWR019
 U 1 1 5FCF7CBC
 P 6900 6000
@@
 $EndComp
 $Comp
-L pcb1-rescue:+3.3V-power #PWR04
+L pcb1-rescue:+3.3V-power-pcb1-rescue #PWR04
 U 1 1 5FCF8D37
 P 2500 3750
@@
 	2000 3750 2500 3750
 $Comp
-L pcb1-rescue:+3.3V-power #PWR013
+L pcb1-rescue:+3.3V-power-pcb1-rescue #PWR013
 U 1 1 5FCFDEDB
 P 5650 5300
@@
 $EndComp
 $Comp
-L pcb1-rescue:+3.3V-power #PWR020
+L pcb1-rescue:+3.3V-power-pcb1-rescue #PWR020
 U 1 1 5FCFEEFD
 P 7350 5100
@@
 $EndComp
 $Comp
-L pcb1-rescue:GND-power #PWR07
+L pcb1-rescue:GND-power-pcb1-rescue #PWR07
 U 1 1 5EAB3202
 P 3550 850
@@
 	3250 1250 3250 1350
 $Comp
-L pcb1-rescue:GND-power #PWR08
+L pcb1-rescue:GND-power-pcb1-rescue #PWR08
 U 1 1 5FD31373
 P 4350 3050
@@
 	5450 6900 5550 6900
 $Comp
-L pcb1-rescue:GND-power #PWR09
+L pcb1-rescue:GND-power-pcb1-rescue #PWR09
 U 1 1 5FD765F3
 P 4500 5500
@@
 $EndComp
 $Comp
-L pcb1-rescue:+3.3V-power #PWR010
+L pcb1-rescue:+3.3V-power-pcb1-rescue #PWR010
 U 1 1 5FD79B08
 P 4500 5600
